File: kicad/Power.kicad_sch (KiCad schematic)
At the start: 17 parts

Commit message: Add files via upload
Parts:
- D29, D44: value (none) -> 74LS32; footprint (none) -> Package_DIP:DIP-14_W7.62mm_Socket
- D35, D85: value (none) -> 74LS08; footprint (none) -> Package_DIP:DIP-14_W7.62mm_Socket
- D36, D42, D73: value (none) -> 74LS04; footprint (none) -> Package_DIP:DIP-14_W7.62mm_Socket
- D40, D57, D66, D71, D77: value (none) -> 74LS74; footprint (none) -> Package_DIP:DIP-14_W7.62mm_Socket
- D41, D75, D78: value (none) -> 74LS00; footprint (none) -> Package_DIP:DIP-14_W7.62mm_Socket
- D43: value (none) -> 74LS33; footprint (none) -> Package_DIP:DIP-14_W7.62mm_Socket
- D76: value (none) -> 74LS05; footprint (none) -> Package_DIP:DIP-14_W7.62mm_Socket
Changed lines of the file:
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@@
       (effects (font (size 1.524 1.524)))
     )
-    (property "Value" "" (id 1) (at 38.735 83.82 0))
-    (property "Footprint" "" (id 2) (at 38.735 82.55 0)
+    (property "Value" "74LS00" (id 1) (at 38.735 83.82 0))
+    (property "Footprint" "Package_DIP:DIP-14_W7.62mm_Socket" (id 2) (at 38.735 82.55 0)
       (effects (font (size 1.27 1.27)) hide)
     )
@@
       (effects (font (size 1.524 1.524)))
     )
-    (property "Value" "" (id 1) (at 224.155 41.275 0))
-    (property "Footprint" "" (id 2) (at 224.155 37.465 0)
+    (property "Value" "74LS04" (id 1) (at 224.155 41.275 0))
+    (property "Footprint" "Package_DIP:DIP-14_W7.62mm_Socket" (id 2) (at 224.155 37.465 0)
       (effects (font (size 1.27 1.27)) hide)
     )
@@
       (effects (font (size 1.524 1.524)))
     )
-    (property "Value" "" (id 1) (at 64.77 128.27 0))
-    (property "Footprint" "" (id 2) (at 64.77 127 0)
+    (property "Value" "74LS00" (id 1) (at 64.77 128.27 0))
+    (property "Footprint" "Package_DIP:DIP-14_W7.62mm_Socket" (id 2) (at 64.77 127 0)
       (effects (font (size 1.27 1.27)) hide)
     )
@@
       (effects (font (size 1.524 1.524)))
     )
-    (property "Value" "" (id 1) (at 25.4 128.27 0))
-    (property "Footprint" "" (id 2) (at 25.4 127 0)
+    (property "Value" "74LS04" (id 1) (at 25.4 128.27 0))
+    (property "Footprint" "Package_DIP:DIP-14_W7.62mm_Socket" (id 2) (at 25.4 127 0)
       (effects (font (size 1.27 1.27)) hide)
     )
@@
       (effects (font (size 1.524 1.524)))
     )
-    (property "Value" "" (id 1) (at 25.4 39.37 0)
-      (effects (font (size 1.524 1.524)))
-    )
-    (property "Footprint" "" (id 2) (at 25.4 38.735 0)
+    (property "Value" "74LS32" (id 1) (at 25.4 39.37 0)
+      (effects (font (size 1.524 1.524)))
+    )
+    (property "Footprint" "Package_DIP:DIP-14_W7.62mm_Socket" (id 2) (at 25.4 38.735 0)
       (effects (font (size 1.27 1.27)) hide)
     )
@@
       (effects (font (size 1.524 1.524)))
     )
-    (property "Value" "" (id 1) (at 218.44 85.725 0)
-      (effects (font (size 1.524 1.524)))
-    )
-    (property "Footprint" "" (id 2) (at 218.44 84.455 0)
+    (property "Value" "74LS74" (id 1) (at 218.44 85.725 0)
+      (effects (font (size 1.524 1.524)))
+    )
+    (property "Footprint" "Package_DIP:DIP-14_W7.62mm_Socket" (id 2) (at 218.44 84.455 0)
       (effects (font (size 1.27 1.27)) hide)
     )
@@
       (effects (font (size 1.524 1.524)))
     )
-    (property "Value" "" (id 1) (at 210.82 41.275 0))
-    (property "Footprint" "" (id 2) (at 210.82 37.465 0)
+    (property "Value" "74LS05" (id 1) (at 210.82 41.275 0))
+    (property "Footprint" "Package_DIP:DIP-14_W7.62mm_Socket" (id 2) (at 210.82 37.465 0)
       (effects (font (size 1.27 1.27)) hide)
     )
@@
       (effects (font (size 1.524 1.524)))
     )
-    (property "Value" "" (id 1) (at 190.5 85.725 0)
-      (effects (font (size 1.524 1.524)))
-    )
-    (property "Footprint" "" (id 2) (at 190.5 84.455 0)
+    (property "Value" "74LS74" (id 1) (at 190.5 85.725 0)
+      (effects (font (size 1.524 1.524)))
+    )
+    (property "Footprint" "Package_DIP:DIP-14_W7.62mm_Socket" (id 2) (at 190.5 84.455 0)
       (effects (font (size 1.27 1.27)) hide)
     )
@@
       (effects (font (size 1.524 1.524)))
     )
-    (property "Value" "" (id 1) (at 83.82 127.635 0)
-      (effects (font (size 1.524 1.524)))
-    )
-    (property "Footprint" "" (id 2) (at 83.82 126.365 0)
+    (property "Value" "74LS74" (id 1) (at 83.82 127.635 0)
+      (effects (font (size 1.524 1.524)))
+    )
+    (property "Footprint" "Package_DIP:DIP-14_W7.62mm_Socket" (id 2) (at 83.82 126.365 0)
       (effects (font (size 1.27 1.27)) hide)
     )
@@
       (effects (font (size 1.524 1.524)))
     )
-    (property "Value" "" (id 1) (at 39.37 40.005 0)
-      (effects (font (size 1.524 1.524)))
-    )
-    (property "Footprint" "" (id 2) (at 39.37 38.735 0)
+    (property "Value" "74LS74" (id 1) (at 39.37 40.005 0)
+      (effects (font (size 1.524 1.524)))
+    )
+    (property "Footprint" "Package_DIP:DIP-14_W7.62mm_Socket" (id 2) (at 39.37 38.735 0)
       (effects (font (size 1.27 1.27)) hide)
     )
@@
       (effects (font (size 1.524 1.524)))
     )
-    (property "Value" "" (id 1) (at 66.675 40.005 0))
-    (property "Footprint" "" (id 2) (at 66.675 38.735 0)
+    (property "Value" "74LS08" (id 1) (at 66.675 40.005 0))
+    (property "Footprint" "Package_DIP:DIP-14_W7.62mm_Socket" (id 2) (at 66.675 38.735 0)
       (effects (font (size 1.27 1.27)) hide)
     )
@@
       (effects (font (size 1.524 1.524)))
     )
-    (property "Value" "" (id 1) (at 25.4 83.82 0)
-      (effects (font (size 1.524 1.524)))
-    )
-    (property "Footprint" "" (id 2) (at 25.4 82.55 0)
+    (property "Value" "74LS04" (id 1) (at 25.4 83.82 0)
+      (effects (font (size 1.524 1.524)))
+    )
+    (property "Footprint" "Package_DIP:DIP-14_W7.62mm_Socket" (id 2) (at 25.4 82.55 0)
       (effects (font (size 1.27 1.27)) hide)
     )
@@
       (effects (font (size 1.524 1.524)))
     )
-    (property "Value" "" (id 1) (at 45.085 128.27 0))
-    (property "Footprint" "" (id 2) (at 45.085 127 0)
+    (property "Value" "74LS00" (id 1) (at 45.085 128.27 0))
+    (property "Footprint" "Package_DIP:DIP-14_W7.62mm_Socket" (id 2) (at 45.085 127 0)
       (effects (font (size 1.27 1.27)) hide)
     )
@@
       (effects (font (size 1.524 1.524)))
     )
-    (property "Value" "" (id 1) (at 52.705 40.005 0))
-    (property "Footprint" "" (id 2) (at 52.705 38.735 0)
+    (property "Value" "74LS33" (id 1) (at 52.705 40.005 0))
+    (property "Footprint" "Package_DIP:DIP-14_W7.62mm_Socket" (id 2) (at 52.705 38.735 0)
       (effects (font (size 1.27 1.27)) hide)
     )
@@
       (effects (font (size 1.27 1.27)) (justify left))
     )
-    (property "Value" "" (id 1) (at 234.95 38.735 0)
+    (property "Value" "74LS74" (id 1) (at 234.95 38.735 0)
       (effects (font (size 1.27 1.27)) (justify left))
     )
-    (property "Footprint" "" (id 2) (at 238.125 37.465 0)
+    (property "Footprint" "Package_DIP:DIP-14_W7.62mm_Socket" (id 2) (at 238.125 37.465 0)
       (effects (font (size 1.27 1.27)) hide)
     )
@@
       (effects (font (size 1.524 1.524)))
     )
-    (property "Value" "" (id 1) (at 204.47 85.725 0))
-    (property "Footprint" "" (id 2) (at 204.47 84.455 0)
+    (property "Value" "74LS32" (id 1) (at 204.47 85.725 0))
+    (property "Footprint" "Package_DIP:DIP-14_W7.62mm_Socket" (id 2) (at 204.47 84.455 0)
       (effects (font (size 1.27 1.27)) hide)
     )
@@
       (effects (font (size 1.524 1.524)))
     )
-    (property "Value" "" (id 1) (at 197.485 38.735 0))
-    (property "Footprint" "" (id 2) (at 197.485 37.465 0)
-      (effects (font (size 1.27 1.27)) hide)
-    )
+    (property "Value" "74LS08" (id 1) (at 197.485 38.735 0))
+    (property "Footprint" "Package_DIP:DIP-14_W7.62mm_Socket" (id 2) (at 197.485 37.465 0)
+      (effects (font (size 1.27 1.27)) hide)
+    )
