File: kicad/clkcrtc.kicad_sch (KiCad schematic)
At the start: 27 parts

Commit message: Add files via upload
Parts:
- C1, C2: value (none) -> 470; footprint (none) -> Common_Alessio:C_Disc_D7.5_P2.5
- C3: value (none) -> CAP; footprint (none) -> Common_Alessio:C_Disc_D7.5_P2.5
- C7: value (none) -> 0,33мк; footprint (none) -> Common_Alessio:C_Disc_D7.5_P2.5
- C8: value (none) -> 1н; footprint (none) -> Common_Alessio:C_Disc_D7.5_P2.5
- D25: value (none) -> MC6845P; footprint (none) -> Package_DIP:DIP-40_W15.24mm_Socket
- D36: value (none) -> 74LS04; footprint (none) -> Package_DIP:DIP-14_W7.62mm_Socket
- D37: value (none) -> 74LS161; footprint (none) -> Package_DIP:DIP-16_W7.62mm_Socket
- D38: value (none) -> 74LS257; footprint (none) -> Package_DIP:DIP-16_W7.62mm_Socket
- D39: value (none) -> 74LS194; footprint (none) -> Package_DIP:DIP-16_W7.62mm_Socket
- D41, D78: value (none) -> 74LS00; footprint (none) -> Package_DIP:DIP-14_W7.62mm_Socket
- D65: value (none) -> 2716; footprint (none) -> Package_DIP:DIP-24_W15.24mm_Socket
- D77: value (none) -> 74LS74; footprint (none) -> Package_DIP:DIP-14_W7.62mm_Socket
- IC63, IC64: value (none) -> MC14520BDP; footprint (none) -> Package_DIP:DIP-16_W7.62mm_Socket
- Q1: value (none) -> 16 MHz; footprint (none) -> Crystal:Crystal_HC49-U_Horizontal
- Q2: value (none) -> 13.333 MHz; footprint (none) -> Crystal:Crystal_HC49-U_Horizontal
- R1, R2, R3, R4: value (none) -> 1,2к; footprint (none) -> Resistor_THT:R_Axial_DIN0204_L3.6mm_D1.6mm_P7.62mm_Horizontal
- R26: value (none) -> 10k; footprint (none) -> Resistor_THT:R_Axial_DIN0204_L3.6mm_D1.6mm_P7.62mm_Horizontal
- R27: value (none) -> 10к; footprint (none) -> Resistor_THT:R_Axial_DIN0204_L3.6mm_D1.6mm_P7.62mm_Horizontal
- R5: value (none) -> 2,7к; footprint (none) -> Resistor_THT:R_Axial_DIN0204_L3.6mm_D1.6mm_P7.62mm_Horizontal
- VD1, VD5: value (none) -> Diode; footprint (none) -> Diode_THT:D_DO-35_SOD27_P7.62mm_Horizontal
