File: kicad/cpu.kicad_sch (KiCad schematic)
At the start: 16 parts

Commit message: Add files via upload
Parts:
- C24: value (none) -> 1мк; footprint (none) -> Capacitors_ThroughHole:C_Radial_D5_L6_P2.5
- D29: value (none) -> 74LS32; footprint (none) -> Package_DIP:DIP-14_W7.62mm_Socket
- D30: value (none) -> Z80; footprint (none) -> Package_DIP:DIP-40_W15.24mm_Socket
- D31: value (none) -> 27512; footprint (none) -> Package_DIP:DIP-28_W15.24mm_Socket
- D35, D85: value (none) -> 74LS08; footprint (none) -> Package_DIP:DIP-14_W7.62mm_Socket
- D43: value (none) -> 74LS33; footprint (none) -> Package_DIP:DIP-14_W7.62mm_Socket
- D66: value (none) -> 74LS74; footprint (none) -> Package_DIP:DIP-14_W7.62mm_Socket
- D67: value (none) -> AM27S20; footprint (none) -> Package_DIP:DIP-16_W7.62mm_Socket
- R135: value (none) -> 10к; footprint (none) -> Resistor_THT:R_Axial_DIN0204_L3.6mm_D1.6mm_P7.62mm_Horizontal
- R14, R15, R25: value (none) -> 2,7к; footprint (none) -> Resistor_THT:R_Axial_DIN0204_L3.6mm_D1.6mm_P7.62mm_Horizontal
- RN2: value (none) -> 10k; footprint (none) -> Resistor_THT:R_Array_SIP4
- RN3: value (none) -> 10k; footprint (none) -> Resistor_THT:R_Array_SIP9
- RN5: value (none) -> 1.2k; footprint (none) -> Resistor_THT:R_Array_SIP5
Changed lines of the file:
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@@
     (in_bom yes) (on_board yes)
     (property "Reference" "R135" (id 0) (at 63.5 94.615 0))
-    (property "Value" "" (id 1) (at 63.5 99.695 0))
-    (property "Footprint" "" (id 2) (at 63.5 98.425 0)
+    (property "Value" "10к" (id 1) (at 63.5 99.695 0))
+    (property "Footprint" "Resistor_THT:R_Axial_DIN0204_L3.6mm_D1.6mm_P7.62mm_Horizontal" (id 2) (at 63.5 98.425 0)
       (effects (font (size 1.524 1.524)) hide)
     )
@@
     (in_bom yes) (on_board yes)
     (property "Reference" "C24" (id 0) (at 67.945 102.235 0))
-    (property "Value" "" (id 1) (at 74.295 102.235 0))
-    (property "Footprint" "" (id 2) (at 72.39 102.235 0)
+    (property "Value" "1мк" (id 1) (at 74.295 102.235 0))
+    (property "Footprint" "Capacitors_ThroughHole:C_Radial_D5_L6_P2.5" (id 2) (at 72.39 102.235 0)
       (effects (font (size 1.524 1.524)) hide)
     )
@@
       (effects (font (size 1.524 1.524)))
     )
-    (property "Value" "" (id 1) (at 49.53 52.705 0))
-    (property "Footprint" "" (id 2) (at 48.895 43.815 0)
+    (property "Value" "Z80" (id 1) (at 49.53 52.705 0))
+    (property "Footprint" "Package_DIP:DIP-40_W15.24mm_Socket" (id 2) (at 48.895 43.815 0)
       (effects (font (size 1.27 1.27)) hide)
     )
@@
       (effects (font (size 1.524 1.524)))
     )
-    (property "Value" "" (id 1) (at 106.68 29.21 0)
-      (effects (font (size 1.524 1.524)))
-    )
-    (property "Footprint" "" (id 2) (at 106.68 22.86 0)
+    (property "Value" "74LS32" (id 1) (at 106.68 29.21 0)
+      (effects (font (size 1.524 1.524)))
+    )
+    (property "Footprint" "Package_DIP:DIP-14_W7.62mm_Socket" (id 2) (at 106.68 22.86 0)
       (effects (font (size 1.27 1.27)) hide)
     )
@@
       (effects (font (size 1.524 1.524)))
     )
-    (property "Value" "" (id 1) (at 106.68 41.91 0)
-      (effects (font (size 1.524 1.524)))
-    )
-    (property "Footprint" "" (id 2) (at 106.68 35.56 0)
+    (property "Value" "74LS32" (id 1) (at 106.68 41.91 0)
+      (effects (font (size 1.524 1.524)))
+    )
+    (property "Footprint" "Package_DIP:DIP-14_W7.62mm_Socket" (id 2) (at 106.68 35.56 0)
       (effects (font (size 1.27 1.27)) hide)
     )
@@
       (effects (font (size 1.524 1.524)))
     )
-    (property "Value" "" (id 1) (at 51.435 133.35 0))
-    (property "Footprint" "" (id 2) (at -2.54 111.125 0)
+    (property "Value" "27512" (id 1) (at 51.435 133.35 0))
+    (property "Footprint" "Package_DIP:DIP-28_W15.24mm_Socket" (id 2) (at -2.54 111.125 0)
       (effects (font (size 1.524 1.524)) hide)
     )
@@
       (effects (font (size 1.524 1.524)))
     )
-    (property "Value" "" (id 1) (at 40.64 183.515 0))
-    (property "Footprint" "" (id 2) (at 40.64 177.165 0)
+    (property "Value" "74LS08" (id 1) (at 40.64 183.515 0))
+    (property "Footprint" "Package_DIP:DIP-14_W7.62mm_Socket" (id 2) (at 40.64 177.165 0)
       (effects (font (size 1.27 1.27)) hide)
     )
@@
       (effects (font (size 1.524 1.524)))
     )
-    (property "Value" "" (id 1) (at 40.64 196.215 0))
-    (property "Footprint" "" (id 2) (at 40.64 189.865 0)
+    (property "Value" "74LS08" (id 1) (at 40.64 196.215 0))
+    (property "Footprint" "Package_DIP:DIP-14_W7.62mm_Socket" (id 2) (at 40.64 189.865 0)
       (effects (font (size 1.27 1.27)) hide)
     )
@@
     (in_bom yes) (on_board yes)
     (property "Reference" "R25" (id 0) (at 45.72 161.925 0))
-    (property "Value" "" (id 1) (at 45.72 167.005 0))
-    (property "Footprint" "" (id 2) (at 45.72 165.735 0)
+    (property "Value" "2,7к" (id 1) (at 45.72 167.005 0))
+    (property "Footprint" "Resistor_THT:R_Axial_DIN0204_L3.6mm_D1.6mm_P7.62mm_Horizontal" (id 2) (at 45.72 165.735 0)
       (effects (font (size 1.524 1.524)) hide)
     )
@@
       (effects (font (size 1.524 1.524)))
     )
-    (property "Value" "" (id 1) (at 119.38 62.865 0))
-    (property "Footprint" "" (id 2) (at 125.73 40.64 0)
+    (property "Value" "AM27S20" (id 1) (at 119.38 62.865 0))
+    (property "Footprint" "Package_DIP:DIP-16_W7.62mm_Socket" (id 2) (at 125.73 40.64 0)
       (effects (font (size 1.27 1.27)) (justify left) hide)
     )
@@
     (in_bom yes) (on_board yes)
     (property "Reference" "R14" (id 0) (at 96.52 76.2 0))
-    (property "Value" "" (id 1) (at 99.06 76.2 0))
-    (property "Footprint" "" (id 2) (at 100.33 76.2 0)
+    (property "Value" "2,7к" (id 1) (at 99.06 76.2 0))
+    (property "Footprint" "Resistor_THT:R_Axial_DIN0204_L3.6mm_D1.6mm_P7.62mm_Horizontal" (id 2) (at 100.33 76.2 0)
       (effects (font (size 1.524 1.524)) hide)
     )
@@
       (effects (font (size 1.524 1.524)))
     )
-    (property "Value" "" (id 1) (at 122.555 109.855 0)
-      (effects (font (size 1.524 1.524)))
-    )
-    (property "Footprint" "" (id 2) (at 111.76 104.14 0)
+    (property "Value" "74LS74" (id 1) (at 122.555 109.855 0)
+      (effects (font (size 1.524 1.524)))
+    )
+    (property "Footprint" "Package_DIP:DIP-14_W7.62mm_Socket" (id 2) (at 111.76 104.14 0)
       (effects (font (size 1.27 1.27)) hide)
     )
@@
       (effects (font (size 1.524 1.524)))
     )
-    (property "Value" "" (id 1) (at 121.92 132.715 0)
-      (effects (font (size 1.524 1.524)))
-    )
-    (property "Footprint" "" (id 2) (at 111.76 127 0)
+    (property "Value" "74LS74" (id 1) (at 121.92 132.715 0)
+      (effects (font (size 1.524 1.524)))
+    )
+    (property "Footprint" "Package_DIP:DIP-14_W7.62mm_Socket" (id 2) (at 111.76 127 0)
       (effects (font (size 1.27 1.27)) hide)
     )
@@
     (in_bom yes) (on_board yes)
     (property "Reference" "R15" (id 0) (at 129.54 121.92 0))
-    (property "Value" "" (id 1) (at 129.54 127 0))
-    (property "Footprint" "" (id 2) (at 129.54 125.73 0)
+    (property "Value" "2,7к" (id 1) (at 129.54 127 0))
+    (property "Footprint" "Resistor_THT:R_Axial_DIN0204_L3.6mm_D1.6mm_P7.62mm_Horizontal" (id 2) (at 129.54 125.73 0)
       (effects (font (size 1.524 1.524)) hide)
     )
@@
       (effects (font (size 1.524 1.524)))
     )
-    (property "Value" "" (id 1) (at 119.38 160.02 0))
-    (property "Footprint" "" (id 2) (at 111.76 157.48 0)
+    (property "Value" "74LS08" (id 1) (at 119.38 160.02 0))
+    (property "Footprint" "Package_DIP:DIP-14_W7.62mm_Socket" (id 2) (at 111.76 157.48 0)
       (effects (font (size 1.27 1.27)) hide)
     )
@@
       (effects (font (size 1.524 1.524)))
     )
-    (property "Value" "" (id 1) (at 142.24 156.21 0))
-    (property "Footprint" "" (id 2) (at 142.24 149.86 0)
+    (property "Value" "74LS33" (id 1) (at 142.24 156.21 0))
+    (property "Footprint" "Package_DIP:DIP-14_W7.62mm_Socket" (id 2) (at 142.24 149.86 0)
       (effects (font (size 1.27 1.27)) hide)
     )
@@
       (effects (font (size 1.524 1.524)))
     )
-    (property "Value" "" (id 1) (at 119.38 147.32 0))
-    (property "Footprint" "" (id 2) (at 111.76 144.78 0)
+    (property "Value" "74LS32" (id 1) (at 119.38 147.32 0))
+    (property "Footprint" "Package_DIP:DIP-14_W7.62mm_Socket" (id 2) (at 111.76 144.78 0)
       (effects (font (size 1.27 1.27)) hide)
     )
@@
       (effects (font (size 1.27 1.27)) (justify left))
     )
-    (property "Value" "" (id 1) (at 139.7 52.705 90)
+    (property "Value" "1.2k" (id 1) (at 139.7 52.705 90)
       (effects (font (size 1.27 1.27)) (justify left))
     )
-    (property "Footprint" "" (id 2) (at 137.668 50.8 90)
+    (property "Footprint" "Resistor_THT:R_Array_SIP5" (id 2) (at 137.668 50.8 90)
       (effects (font (size 1.27 1.27)) hide)
     )
@@
       (effects (font (size 1.27 1.27)) (justify right))
     )
-    (property "Value" "" (id 1) (at 134.62 74.93 90)
+    (property "Value" "1.2k" (id 1) (at 134.62 74.93 90)
       (effects (font (size 1.27 1.27)) (justify right))
     )
-    (property "Footprint" "" (id 2) (at 136.652 73.025 90)
+    (property "Footprint" "Resistor_THT:R_Array_SIP5" (id 2) (at 136.652 73.025 90)
       (effects (font (size 1.27 1.27)) hide)
     )
@@
     (in_bom yes) (on_board yes) (fields_autoplaced)
     (property "Reference" "RN2" (id 0) (at 182.626 16.51 90))
-    (property "Value" "" (id 1) (at 182.626 19.05 90))
-    (property "Footprint" "" (id 2) (at 182.88 32.385 90)
+    (property "Value" "10k" (id 1) (at 182.626 19.05 90))
+    (property "Footprint" "Resistor_THT:R_Array_SIP4" (id 2) (at 182.88 32.385 90)
       (effects (font (size 1.27 1.27)) hide)
     )
@@
       (effects (font (size 1.27 1.27)) (justify right))
     )
-    (property "Value" "" (id 1) (at 139.7 74.93 90)
+    (property "Value" "1.2k" (id 1) (at 139.7 74.93 90)
       (effects (font (size 1.27 1.27)) (justify right))
     )
-    (property "Footprint" "" (id 2) (at 141.732 73.025 90)
+    (property "Footprint" "Resistor_THT:R_Array_SIP5" (id 2) (at 141.732 73.025 90)
       (effects (font (size 1.27 1.27)) hide)
     )
@@
       (effects (font (size 1.27 1.27)) (justify left))
     )
-    (property "Value" "" (id 1) (at 134.62 52.705 90)
+    (property "Value" "1.2k" (id 1) (at 134.62 52.705 90)
       (effects (font (size 1.27 1.27)) (justify left))
     )
-    (property "Footprint" "" (id 2) (at 132.588 50.8 90)
+    (property "Footprint" "Resistor_THT:R_Array_SIP5" (id 2) (at 132.588 50.8 90)
       (effects (font (size 1.27 1.27)) hide)
     )
@@
     (in_bom yes) (on_board yes) (fields_autoplaced)
     (property "Reference" "RN3" (id 0) (at 182.626 33.655 90))
-    (property "Value" "" (id 1) (at 182.626 36.195 90))
-    (property "Footprint" "" (id 2) (at 182.88 62.865 90)
-      (effects (font (size 1.27 1.27)) hide)
-    )
+    (property "Value" "10k" (id 1) (at 182.626 36.195 90))
+    (property "Footprint" "Resistor_THT:R_Array_SIP9" (id 2) (at 182.88 62.865 90)
+      (effects (font (size 1.27 1.27)) hide)
+    )
