File: kicad/fdc.kicad_sch (KiCad schematic)
At the start: 15 parts

Commit message: Add files via upload
Parts:
- C18: value (none) -> CAP; footprint (none) -> MyLib_metric:C_Disc_D7.5_P2.5
- D68: value (none) -> 74LS174; footprint (none) -> Package_DIP:DIP-16_W7.62mm_Socket
- D69: value (none) -> 27S18; footprint (none) -> Package_DIP:DIP-16_W7.62mm_Socket
- D70: value (none) -> UPD765AC; footprint (none) -> Package_DIP:DIP-40_W15.24mm_Socket
- D71: value (none) -> 74LS74; footprint (none) -> Package_DIP:DIP-14_W7.62mm_Socket
- D72: value (none) -> 74LS93; footprint (none) -> Package_DIP:DIP-14_W7.62mm_Socket
- D73: value (none) -> 74LS04; footprint (none) -> Package_DIP:DIP-14_W7.62mm_Socket
- D74: value (none) -> 74LS155; footprint (none) -> Package_DIP:DIP-16_W7.62mm_Socket
- D75: value (none) -> 74LS00; footprint (none) -> Package_DIP:DIP-14_W7.62mm_Socket
- D76: value (none) -> 74LS05; footprint (none) -> Package_DIP:DIP-14_W7.62mm_Socket
- D85: value (none) -> 74LS08; footprint (none) -> Package_DIP:DIP-14_W7.62mm_Socket
- R76: value (none) -> 2,7к; footprint (none) -> Resistor_THT:R_Axial_DIN0204_L3.6mm_D1.6mm_P7.62mm_Horizontal
- RN8: value (none) -> 2,7k; footprint (none) -> Resistor_THT:R_Array_SIP5
- RN9: value (none) -> 1.2k; footprint (none) -> Resistor_THT:R_Array_SIP6
- X4: value (none) -> SLOT-34; footprint (none) -> Common_Alessio:SLOT-34
