File: kicad/gatearray.kicad_sch (KiCad schematic)
At the start: 64 parts

Commit message: Add files via upload
Parts:
- C14: value (none) -> 100мк; footprint (none) -> Capacitors_ThroughHole:C_Radial_D5_L6_P2.5
- C15, C16, C17, C4, C5: value (none) -> CAP; footprint (none) -> Common_Alessio:C_Disc_D7.5_P2.5
- D26: value (none) -> 74LS253; footprint (none) -> Package_DIP:DIP-16_W7.62mm_Socket
- D28: value (none) -> AM27S20; footprint (none) -> Package_DIP:DIP-16_W7.62mm_Socket
- D29, D44: value (none) -> 74LS32; footprint (none) -> Package_DIP:DIP-14_W7.62mm_Socket
- D32, D55, D56, D59: value (none) -> 74LS174; footprint (none) -> Package_DIP:DIP-16_W7.62mm_Socket
- D35, D85: value (none) -> 74LS08; footprint (none) -> Package_DIP:DIP-14_W7.62mm_Socket
- D43: value (none) -> 74LS33; footprint (none) -> Package_DIP:DIP-14_W7.62mm_Socket
- D49, D50, D51: value (none) -> 74LS194; footprint (none) -> Package_DIP:DIP-16_W7.62mm_Socket
- D52, D53: value (none) -> 74LS153; footprint (none) -> Package_DIP:DIP-16_W7.62mm_Socket
- D54: value (none) -> 74LS155; footprint (none) -> Package_DIP:DIP-16_W7.62mm_Socket
- D57, D77: value (none) -> 74LS74; footprint (none) -> Package_DIP:DIP-14_W7.62mm_Socket
- D58: value (none) -> 74LS374; footprint (none) -> Package_DIP:DIP-20_W7.62mm_Socket
- D60, D61: value (none) -> 1802ИР1; footprint (none) -> MyLib_metric:DIP-24
- D62: value (none) -> 2716; footprint (none) -> Package_DIP:DIP-24_W15.24mm_Socket
- D87, D88: value (none) -> 74LS170; footprint (none) -> Package_DIP:DIP-16_W7.62mm_Socket
- D89: value (none) -> 74LS245; footprint (none) -> Package_DIP:DIP-20_W7.62mm_Socket
- DR1: value (none) -> 91мкГ; footprint (none) -> Inductor_THT:L_Axial_L9.5mm_D4.0mm_P15.24mm_Horizontal_Fastron_SMCC
- R101, R134, R16, R53, R55, R57: value (none) -> 360; footprint (none) -> Resistor_THT:R_Axial_DIN0204_L3.6mm_D1.6mm_P7.62mm_Horizontal
- R136: value (none) -> RES; footprint (none) -> Resistor_THT:R_Axial_DIN0204_L3.6mm_D1.6mm_P7.62mm_Horizontal
- R51, R60: value (none) -> 1,2к; footprint (none) -> Resistor_THT:R_Axial_DIN0204_L3.6mm_D1.6mm_P7.62mm_Horizontal
- R52, R54, R56: value (none) -> 200; footprint (none) -> Resistor_THT:R_Axial_DIN0204_L3.6mm_D1.6mm_P7.62mm_Horizontal
- R58: value (none) -> 510; footprint (none) -> Resistor_THT:R_Axial_DIN0204_L3.6mm_D1.6mm_P7.62mm_Horizontal
- R59: value (none) -> 6,8к; footprint (none) -> Resistor_THT:R_Axial_DIN0204_L3.6mm_D1.6mm_P7.62mm_Horizontal
- R6: value (none) -> 2,7к; footprint (none) -> Resistor_THT:R_Axial_DIN0204_L3.6mm_D1.6mm_P7.62mm_Horizontal
- R61: value (none) -> 3,3к; footprint (none) -> Resistor_THT:R_Axial_DIN0204_L3.6mm_D1.6mm_P7.62mm_Horizontal
- R62, R63, R64, R66, R81: value (none) -> 220; footprint (none) -> Resistor_THT:R_Axial_DIN0204_L3.6mm_D1.6mm_P7.62mm_Horizontal
- R65: value (none) -> 120; footprint (none) -> Resistor_THT:R_Axial_DIN0204_L3.6mm_D1.6mm_P7.62mm_Horizontal
- RN6: value (none) -> 1.2k; footprint (none) -> Resistor_THT:R_Array_SIP5
- RN7: value (none) -> 1.2k; footprint (none) -> Resistor_THT:R_Array_SIP6
- VD12, VD2, VD8: value (none) -> Diode; footprint (none) -> Diode_THT:D_DO-35_SOD27_P7.62mm_Horizontal
- VD15: value (none) -> CAPS; footprint (none) -> Connector_PinHeader_2.00mm:PinHeader_1x02_P2.00mm_Vertical
- VD3: value (none) -> DA; footprint (none) -> Connector_PinHeader_2.00mm:PinHeader_1x02_P2.00mm_Vertical
- X2: value (none) -> CONN-7S; footprint (none) -> Common_Alessio:DNR-8F1R
