File: kicad/periph.kicad_sch (KiCad schematic)
At the start: 83 parts

Commit message: Add files via upload
Parts:
- C10, C22: value (none) -> 100мк
- C23: value (none) -> 0,47мк; footprint (none) -> MyLib_metric:C_Disc_D7.5_P2.5
- C25, C26: value (none) -> 47мк
- C6: value (none) -> 1мк
- C9: value (none) -> 1,5мк
Changed lines of the file:
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@@
     (in_bom yes) (on_board yes)
     (property "Reference" "C9" (id 0) (at 123.825 141.605 0))
-    (property "Value" "" (id 1) (at 130.175 141.605 0))
+    (property "Value" "1,5мк" (id 1) (at 130.175 141.605 0))
     (property "Footprint" "" (id 2) (at 128.27 141.605 0)
       (effects (font (size 1.524 1.524)) hide)
@@
     (in_bom yes) (on_board yes)
     (property "Reference" "C10" (id 0) (at 151.765 160.02 0))
-    (property "Value" "" (id 1) (at 158.115 160.02 0))
+    (property "Value" "100мк" (id 1) (at 158.115 160.02 0))
     (property "Footprint" "" (id 2) (at 156.21 160.02 0)
       (effects (font (size 1.524 1.524)) hide)
@@
     (in_bom yes) (on_board yes)
     (property "Reference" "C23" (id 0) (at 230.505 273.685 0))
-    (property "Value" "" (id 1) (at 236.855 273.685 0))
-    (property "Footprint" "" (id 2) (at 234.95 273.685 0)
+    (property "Value" "0,47мк" (id 1) (at 236.855 273.685 0))
+    (property "Footprint" "MyLib_metric:C_Disc_D7.5_P2.5" (id 2) (at 234.95 273.685 0)
       (effects (font (size 1.524 1.524)) hide)
     )
@@
     (in_bom yes) (on_board yes)
     (property "Reference" "C26" (id 0) (at 218.44 241.935 0))
-    (property "Value" "" (id 1) (at 218.44 248.285 0))
+    (property "Value" "47мк" (id 1) (at 218.44 248.285 0))
     (property "Footprint" "" (id 2) (at 218.44 246.38 0)
       (effects (font (size 1.524 1.524)) hide)
@@
     (in_bom yes) (on_board yes)
     (property "Reference" "C25" (id 0) (at 200.025 250.19 0))
-    (property "Value" "" (id 1) (at 206.375 250.19 0))
+    (property "Value" "47мк" (id 1) (at 206.375 250.19 0))
     (property "Footprint" "" (id 2) (at 204.47 250.19 0)
       (effects (font (size 1.524 1.524)) hide)
@@
     (in_bom yes) (on_board yes)
     (property "Reference" "C22" (id 0) (at 198.12 263.525 0))
-    (property "Value" "" (id 1) (at 198.12 269.875 0))
+    (property "Value" "100мк" (id 1) (at 198.12 269.875 0))
     (property "Footprint" "" (id 2) (at 198.12 267.97 0)
       (effects (font (size 1.524 1.524)) hide)
@@
     (in_bom yes) (on_board yes)
     (property "Reference" "C6" (id 0) (at 151.765 185.42 0))
-    (property "Value" "" (id 1) (at 158.115 185.42 0))
+    (property "Value" "1мк" (id 1) (at 158.115 185.42 0))
     (property "Footprint" "" (id 2) (at 156.21 185.42 0)
       (effects (font (size 1.524 1.524)) hide)
