File: kicad/ram.kicad_sch (KiCad schematic)
At the start: 49 parts

Commit message: Add files via upload
Parts:
- D1, D10, D11, D12, D13, D14, D15, D16, D2, D3, D4, D5, D6, D7, D8, D9: value (none) -> HM50256P-20; footprint (none) -> Package_DIP:DIP-16_W7.62mm
- D20, D21, D22, D23: value (none) -> 74LS153; footprint (none) -> Package_DIP:DIP-16_W7.62mm_Socket
- D24: value (none) -> 74LS151; footprint (none) -> Package_DIP:DIP-16_W7.62mm_Socket
- D36, D42: value (none) -> 74LS04; footprint (none) -> Package_DIP:DIP-14_W7.62mm_Socket
- D40: value (none) -> 74LS74; footprint (none) -> Package_DIP:DIP-14_W7.62mm_Socket
- D41, D75: value (none) -> 74LS00; footprint (none) -> Package_DIP:DIP-14_W7.62mm_Socket
- D43: value (none) -> 74LS33; footprint (none) -> Package_DIP:DIP-14_W7.62mm_Socket
- D44: value (none) -> 74LS32; footprint (none) -> Package_DIP:DIP-14_W7.62mm_Socket
- D45, D46, D47, D48: value (none) -> 74LS373; footprint (none) -> Package_DIP:DIP-20_W7.62mm_Socket
- D85: value (none) -> 74LS08; footprint (none) -> Package_DIP:DIP-14_W7.62mm_Socket
- R24, R39, R40, R41, R42, R43, R44, R45, R46, R7, R77, R78, R79, R8, R80, R9: value (none) -> 51; footprint (none) -> Resistor_THT:R_Axial_DIN0204_L3.6mm_D1.6mm_P7.62mm_Horizontal
