File: board/Aleste520v4.kicad_pcb (KiCad board)
At the start: 2 copper layers, 400.9 x 280.5 mm, 334 parts, among them P1 PIN, P2 PIN, P3 PIN, P4 PIN, P5 PIN, P6 PIN, P7 PIN, P8 PIN, Q1 16 MHz, Q2 13.333 MHz, Q3 QUARTZ, U1 HM50256P-20, U10 HM50256P-20, U11 HM50256P-20, U12 HM50256P-20, U13 HM50256P-20, U14 HM50256P-20, U15 HM50256P-20, U16 HM50256P-20, U17 8255, U18 AY-3-8910, U19 MC146818P, U2 HM50256P-20, U20 74LS153, U21 74LS153, U22 74LS153, U23 74LS153, U24 74LS151, U25 MC6845, U26 74LS253, U28 AM27S20, U29 74LS32, U3 HM50256P-20, U30 Z80CPU, U31 27C512, U32 74LS174, U33 8253, U34 8251A, U35 74LS08, U36 74LS04, U37 74LS161, U38 74LS257, U39 74LS194, U4 HM50256P-20, U40 74LS74, U41 74HC00, U42 74LS04, U43 74LS02, U44 74LS32, U45 74LS373, U46 74LS373, U47 74LS373, U48 74LS373, U49 74LS194, U5 HM50256P-20, U50 74LS194, U51 74LS194, U52 74LS153, U53 74LS153, U54 74LS155, U55 74LS174, U56 74LS174, U57 74LS74, U58 74LS374, U59 74LS174, U6 HM50256P-20, U60 AM29705, U61 AM29705, U62 2716, U63 MC14520BCP, U64 MC14520BCP, U65 2716, U66 74LS74, U67 AM27S20, U68 74LS174, U69 SN74188, U7 HM50256P-20, U70 8272, U71 74LS74, U72 74LS93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

Commit message: Reorganize into board/, keyboard/, case/, rom/; upgrade X8/X9 to 2x06 2.54mm; add 11 M3 holes & PicoPSU wiring; add Cherry MX NKRO keyboard & anti-flex OpenSCAD case
Parts:
- added MH1: M3_Mount, MountingHole:MountingHole_3.2mm_M3_Pad, F.Cu at (23.5, 24.0)
- added MH10: M3_Mount, MountingHole:MountingHole_3.2mm_M3_Pad, F.Cu at (283.5, 286.5)
- added MH11: M3_Mount, MountingHole:MountingHole_3.2mm_M3_Pad, F.Cu at (406.5, 256.5)
- added MH2: M3_Mount, MountingHole:MountingHole_3.2mm_M3_Pad, F.Cu at (215.0, 24.0)
- added MH3: M3_Mount, MountingHole:MountingHole_3.2mm_M3_Pad, F.Cu at (273.0, 24.0)
- added MH4: M3_Mount, MountingHole:MountingHole_3.2mm_M3_Pad, F.Cu at (411.5, 24.0)
- added MH5: M3_Mount, MountingHole:MountingHole_3.2mm_M3_Pad, F.Cu at (41.0, 130.0)
- added MH6: M3_Mount, MountingHole:MountingHole_3.2mm_M3_Pad, F.Cu at (220.0, 131.0)
- added MH7: M3_Mount, MountingHole:MountingHole_3.2mm_M3_Pad, F.Cu at (409.5, 148.0)
- added MH8: M3_Mount, MountingHole:MountingHole_3.2mm_M3_Pad, F.Cu at (23.5, 286.5)
- added MH9: M3_Mount, MountingHole:MountingHole_3.2mm_M3_Pad, F.Cu at (148.0, 285.5)
- R37: value 10М -> 10ð£
Routing:
- net GND: vias 3690 -> 3689
