File: board/periph.kicad_sch (KiCad schematic)
At the start: 95 parts, among them P7 PIN, P8 PIN, Q3 QUARTZ, U17 8255, U18 AY-3-8910, U19 MC146818P, U33 8253, U34 8251A, U41 74HC00, U42 74LS04, U75 74HC00, U78 74LS00, U79 74LS174, U80 74LS145, U81 74LS151, U82 AM29705, U83 AM29705, U84 74LS374, U86 SN75150P, X3 CONN-5S, X5.A1 CONN-7S, X5.B1 CONN-7S, X6 CONN-7S, X7 CONN-7S, X8 CONN-12, X9 CONN-12

Commit message: Reorganize into board/, keyboard/, case/, rom/; upgrade X8/X9 to 2x06 2.54mm; add 11 M3 holes & PicoPSU wiring; add Cherry MX NKRO keyboard & anti-flex OpenSCAD case
Parts:
- X8, X9: footprint Connector_PinHeader_1.27mm:PinHeader_1x12_P1.27mm_Vertical -> Connector_PinHeader_2.54mm:PinHeader_2x06_P2.54mm_Vertical
Changed lines of the file:
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@@
       (effects (font (size 1.27 1.27)) hide)
     )
-    (property "Footprint" "Connector_PinHeader_1.27mm:PinHeader_1x12_P1.27mm_Vertical" (at 259.08 29.21 0)
+    (property "Footprint" "Connector_PinHeader_2.54mm:PinHeader_2x06_P2.54mm_Vertical" (at 259.08 29.21 0)
       (effects (font (size 1.524 1.524)) hide)
     )
@@
       (effects (font (size 1.27 1.27)) hide)
     )
-    (property "Footprint" "Connector_PinHeader_1.27mm:PinHeader_1x12_P1.27mm_Vertical" (at 259.08 95.25 0)
+    (property "Footprint" "Connector_PinHeader_2.54mm:PinHeader_2x06_P2.54mm_Vertical" (at 259.08 95.25 0)
       (effects (font (size 1.524 1.524)) hide)
     )
