File: keyboard/Aleste520_Keyboard.kicad_pcb (KiCad board)
At the start: 2 copper layers, 358 x 122 mm, 175 parts, among them J1 X8_COLS_2x06, J2 X9_ROWS_2x06, SW1 ESC, SW10 9, SW11 0, SW12 TAB, SW13 Q, SW14 W, SW15 E, SW16 R, SW17 T, SW18 Y, SW19 U, SW2 1, SW20 I, SW21 O, SW22 P, SW23 CAPS, SW24 A, SW25 S, SW26 D, SW27 F, SW28 G, SW29 H, SW3 2, SW30 J, SW31 K, SW32 L, SW33 SEMI, SW34 SHIFT, SW35 Z, SW36 X, SW37 C, SW38 V, SW39 B, SW4 3, SW40 N, SW41 M, SW42 COMMA, SW43 DOT, SW44 SLASH, SW45 CTRL, SW46 RUS_LAT, SW47 COPY, SW48 STOP, SW49 SELECT, SW5 4, SW50 SPACE, SW51 GRAPH, SW52 CODE, SW53 MINUS, SW54 CARET, SW55 AT, SW56 F0, SW57 F1, SW58 F2, SW59 F3, SW6 5, SW60 F4, SW61 F5, SW62 F6, SW63 F7, SW64 F8, SW65 F9, SW66 FDOT, SW67 ENTER_NP, SW68 LBRACK, SW69 RBRACK, SW7 6, SW70 BSLASH, SW71 COLON, SW72 CLR, SW73 DEL, SW74 INS, SW75 HOME, SW76 END, SW77 UP, SW78 DOWN, SW79 LEFT, SW8 7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

Commit message: Feat(keyboard,case): decode RFVDKEY.BIN/AL512.BIN matrix, redesign staggered keyboard PCB with 6.25U stabilized Spacebar, and convert case to FreeCAD 1.1 (.FCStd)
Parts:
- added D82: 1N4148, Diode_THT:D_DO-35_SOD27_P7.62mm_Horizontal, F.Cu at (215.7, 113.0)
- added SW83: RESET, Button_Switch_Keyboard:SW_Cherry_MX_1.00u_PCB, F.Cu at (339.5, 26.0)
- SW10: value 9 -> DEL; footprint Button_Switch_Keyboard:SW_Cherry_MX_1.00u_PCB -> Button_Switch_Keyboard:SW_Cherry_MX_1.25u_PCB
- SW11: value 0 -> 1
- SW12: value TAB -> 2
- SW13: value Q -> 3
- SW14: value W -> 4
- SW15: value E -> 5
- SW16: value R -> 6
- SW17: value T -> 7
- SW18: value Y -> 8
- SW19: value U -> 9
- SW2: value 1 -> F1_MSX; footprint Button_Switch_Keyboard:SW_Cherry_MX_1.00u_PCB -> Button_Switch_Keyboard:SW_Cherry_MX_1.25u_PCB
- SW20: value I -> 0
- SW21: value O -> MINUS
- SW22: value P -> CARET
- SW23: value CAPS -> BSLASH
- SW24: value A -> F7
- SW25: value S -> F8
- SW26: value D -> F9
- SW27: value F -> UP
- SW28: value G -> TAB; footprint Button_Switch_Keyboard:SW_Cherry_MX_1.00u_PCB -> Button_Switch_Keyboard:SW_Cherry_MX_1.50u_PCB
- SW29: value H -> Q
- SW3: value 2 -> F2_MSX; footprint Button_Switch_Keyboard:SW_Cherry_MX_1.00u_PCB -> Button_Switch_Keyboard:SW_Cherry_MX_1.25u_PCB
- SW30: value J -> W
- SW31: value K -> E
- SW32: value L -> R
- SW33: value SEMI -> T
- SW34: value SHIFT -> Y
- SW35: value Z -> U
- SW36: value X -> I
- SW37: value C -> O
- SW38: value V -> P
- SW39: value B -> AT
- SW4: value 3 -> F3_MSX; footprint Button_Switch_Keyboard:SW_Cherry_MX_1.00u_PCB -> Button_Switch_Keyboard:SW_Cherry_MX_1.25u_PCB
- SW40: value N -> LBRACK
- SW41: value M -> F4
- SW42: value COMMA -> F5
- SW43: value DOT -> F6
- SW44: value SLASH -> LEFT
- SW45: value CTRL -> CAPS; footprint Button_Switch_Keyboard:SW_Cherry_MX_1.00u_PCB -> Button_Switch_Keyboard:SW_Cherry_MX_1.75u_PCB
- SW46: value RUS_LAT -> A
- SW47: value COPY -> S
- SW48: value STOP -> D
- SW49: value SELECT -> F
- SW5: value 4 -> F4_MSX; footprint Button_Switch_Keyboard:SW_Cherry_MX_1.00u_PCB -> Button_Switch_Keyboard:SW_Cherry_MX_1.25u_PCB
- SW50: value SPACE -> G
- SW51: value GRAPH -> H
- SW52: value CODE -> J
- SW53: value MINUS -> K
- SW54: value CARET -> L
- SW55: value AT -> SEMI
- SW56: value F0 -> COLON
- SW57: value F1 -> RBRACK
- SW58: value F2 -> F1
- SW59: value F3 -> F2
- SW6: value 5 -> F5_MSX; footprint Button_Switch_Keyboard:SW_Cherry_MX_1.00u_PCB -> Button_Switch_Keyboard:SW_Cherry_MX_1.25u_PCB
- SW60: value F4 -> F3
- SW61: value F5 -> RIGHT
- SW62: value F6 -> SHIFT; footprint Button_Switch_Keyboard:SW_Cherry_MX_1.00u_PCB -> Button_Switch_Keyboard:SW_Cherry_MX_2.00u_PCB
- SW63: value F7 -> Z
- SW64: value F8 -> X
- SW65: value F9 -> C
- SW66: value FDOT -> V
- SW67: value ENTER_NP -> B
- SW68: value LBRACK -> N
- SW69: value RBRACK -> M
- SW7: value 6 -> SELECT; footprint Button_Switch_Keyboard:SW_Cherry_MX_1.00u_PCB -> Button_Switch_Keyboard:SW_Cherry_MX_1.25u_PCB
- SW70: value BSLASH -> COMMA
- SW71: value COLON -> DOT
- SW72: value CLR -> SLASH
- SW73: value DEL -> RETURN; footprint Button_Switch_Keyboard:SW_Cherry_MX_1.00u_PCB -> Button_Switch_Keyboard:SW_Cherry_MX_1.50u_PCB
- SW74: value INS -> F0
- SW75: value HOME -> FDOT
- SW76: value END -> ENTER
- SW77: value UP -> DOWN
- SW78: value DOWN -> CTRL; footprint Button_Switch_Keyboard:SW_Cherry_MX_1.00u_PCB -> Button_Switch_Keyboard:SW_Cherry_MX_1.50u_PCB
- SW79: value LEFT -> RUS_LAT; footprint Button_Switch_Keyboard:SW_Cherry_MX_1.00u_PCB -> Button_Switch_Keyboard:SW_Cherry_MX_1.25u_PCB
- SW8: value 7 -> STOP; footprint Button_Switch_Keyboard:SW_Cherry_MX_1.00u_PCB -> Button_Switch_Keyboard:SW_Cherry_MX_1.25u_PCB
- SW80: value RIGHT -> COPY; footprint Button_Switch_Keyboard:SW_Cherry_MX_1.00u_PCB -> Button_Switch_Keyboard:SW_Cherry_MX_1.25u_PCB
- SW81: value RETURN -> SPACE; footprint Button_Switch_Keyboard:SW_Cherry_MX_1.00u_PCB -> Button_Switch_Keyboard:SW_Cherry_MX_6.25u_PCB
- SW82: value RESET -> GRAPH; footprint Button_Switch_Keyboard:SW_Cherry_MX_1.00u_PCB -> Button_Switch_Keyboard:SW_Cherry_MX_1.50u_PCB
- SW9: value 8 -> CLR; footprint Button_Switch_Keyboard:SW_Cherry_MX_1.00u_PCB -> Button_Switch_Keyboard:SW_Cherry_MX_1.25u_PCB
- moved SW78 318.3 mm to (24.8, 113.0)
- moved D78 317.6 mm to (17.0, 113.0)
- moved SW79 289.3 mm to (51.0, 113.0)
- moved D79 288.6 mm to (43.1, 113.0)
- moved SW80 263.2 mm to (74.8, 113.0)
- moved D80 262.5 mm to (67.0, 113.0)
- moved SW11 244.4 mm to (20.0, 43.5)
- moved D11 243.7 mm to (12.2, 43.5)
- moved D24 234.5 mm to (273.2, 43.5)
- moved SW24 233.8 mm to (281.0, 43.5)
- moved D25 229.6 mm to (292.2, 43.5)
- moved SW25 228.9 mm to (300.1, 43.5)
- moved D23 226.2 mm to (240.8, 43.5)
- moved SW23 225.5 mm to (248.6, 43.5)
- moved D26 224.7 mm to (311.3, 43.5)
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Connections:
- D1 pad 1: KM0 -> KM1
- D10 pad 1: KM9 -> KM5
- D11 pad 1: KM10 -> KM3
- D12 pad 1: KM0 -> KM4
- D13 pad 1: KM1 -> KM5
- D14 pad 1: KM2 -> KM6
- D15 pad 1: KM3 -> KM7
- D16 pad 1: KM4 -> KM8
- D17 pad 1: KM5 -> KM9
- D18 pad 1: KM6 -> KM10
- D19 pad 1: KM7 -> KM10
- D2 pad 1: KM1 -> KM3
- D20 pad 1: KM8 -> KM9
- D21 pad 1: KM9 -> KM8
- D22 pad 1: KM10 -> KM3
- D23 pad 1: KM0 -> KM9
- D24 pad 1: KM1 -> KM0
- D25 pad 1: KM2 -> KM0
- D26 pad 1: KM3 -> KM0
- D27 pad 1: KM4 -> KM7
- D28 pad 1: KM5 -> KM1
- D29 pad 1: KM6 -> KM2
- D3 pad 1: KM2 -> KM4
- D30 pad 1: KM7 -> KM4
- D31 pad 1: KM8 -> KM6
- D32 pad 1: KM9 -> KM7
- D33 pad 1: KM10 -> KM7
- D34 pad 1: KM0 -> KM3
- D35 pad 1: KM1 -> KM4
- D36 pad 1: KM2 -> KM6
- D37 pad 1: KM3 -> KM8
- D38 pad 1: KM4 -> KM6
- D39 pad 1: KM5 -> KM10
- D4 pad 1: KM3 -> KM5
- D40 pad 1: KM6 -> KM9
- D41 pad 1: KM7 -> KM3
- D42 pad 1: KM8 -> KM3
- D43 pad 1: KM9 -> KM3
- D44 pad 1: KM10 -> KM9
- D45 pad 1: KM0 -> KM1
- D46 pad 1: KM1 -> KM5
- D47 pad 1: KM2 -> KM4
- D48 pad 1: KM3 -> KM10
- D49 pad 1: KM4 -> KM2
- D5 pad 1: KM4 -> KM7
- D50 pad 1: KM5 -> KM8
- D51 pad 1: KM6 -> KM9
- D52 pad 1: KM7 -> KM2
- D53 pad 1: KM8 -> KM5
- D55 pad 1: KM10 -> KM2
- D56 pad 1: KM0 -> KM8
- D57 pad 1: KM1 -> KM10
- D59 pad 1: KM3 -> KM2
- D6 pad 1: KM5 -> KM8
- D60 pad 1: KM4 -> KM2
- D61 pad 1: KM5 -> KM6
- D62 pad 1: KM6 -> KM0
- D63 pad 1: KM7 -> KM10
- D65 pad 1: KM9 -> KM3
- D67 pad 1: KM0 -> KM9
- D68 pad 1: KM1 -> KM7
- D69 pad 1: KM2 -> KM5
- D7 pad 1: KM6 -> KM5
- D70 pad 1: KM3 -> KM10
- D71 pad 1: KM4 -> KM8
- D72 pad 1: KM5 -> KM7
- D74 pad 1: KM7 -> KM1
- D75 pad 1: KM8 -> KM1
- D76 pad 1: KM9 -> KM1
- D77 pad 1: KM0 -> KM7
- D79 pad 1: KM2 -> KM1
- D8 pad 1: KM7 -> KM5
- D80 pad 1: KM3 -> KM2
- D81 pad 1: KM4 -> KM6
- D9 pad 1: KM8 -> KM4
- SW10 pad 2: KM11 -> KM16
- SW11 pad 2: KM11 -> KM12
- SW14 pad 2: KM12 -> KM11
- SW17 pad 2: KM12 -> KM11
- SW18 pad 2: KM12 -> KM11
- SW19 pad 2: KM12 -> KM18
- SW20 pad 2: KM12 -> KM18
- SW21 pad 2: KM12 -> KM18
- SW22 pad 2: KM12 -> KM15
- SW23 pad 2: KM13 -> KM16
- SW24 pad 2: KM13 -> KM16
- SW25 pad 2: KM13 -> KM17
- SW26 pad 2: KM13 -> KM18
- SW27 pad 2: KM13 -> KM17
- SW28 pad 2: KM13 -> KM12
- SW29 pad 2: KM13 -> KM14
- SW30 pad 2: KM13 -> KM14
- SW31 pad 2: KM13 -> KM12
- SW32 pad 2: KM13 -> KM14
- SW33 pad 2: KM13 -> KM15
- SW35 pad 2: KM14 -> KM13
- SW38 pad 2: KM14 -> KM13
- SW40 pad 2: KM14 -> KM12
- SW41 pad 2: KM14 -> KM16
- SW42 pad 2: KM14 -> KM17
- SW43 pad 2: KM14 -> KM18
- SW44 pad 2: KM14 -> KM15
- SW46 pad 2: KM15 -> KM14
- SW48 pad 2: KM15 -> KM13
- SW49 pad 2: KM15 -> KM13
- SW50 pad 2: KM15 -> KM13
- SW51 pad 2: KM15 -> KM17
- SW52 pad 2: KM15 -> KM12
- SW53 pad 2: KM15 -> KM13
- SW54 pad 2: KM15 -> KM13
- SW55 pad 2: KM15 -> KM11
- SW56 pad 2: KM16 -> KM17
- SW57 pad 2: KM16 -> KM12
- SW59 pad 2: KM16 -> KM17
- SW60 pad 2: KM16 -> KM18
- SW62 pad 2: KM16 -> KM15
- SW63 pad 2: KM16 -> KM17
- SW64 pad 2: KM16 -> KM15
- SW65 pad 2: KM16 -> KM13
- SW67 pad 2: KM17 -> KM14
- SW68 pad 2: KM17 -> KM13
- SW69 pad 2: KM17 -> KM15
- SW7 pad 2: KM11 -> KM18
- SW70 pad 2: KM17 -> KM15
- SW71 pad 2: KM17 -> KM16
- SW72 pad 2: KM17 -> KM18
- SW74 pad 2: KM17 -> KM16
- SW76 pad 2: KM17 -> KM18
- SW77 pad 2: KM18 -> KM16
- SW78 pad 2: KM18 -> KM13
- SW79 pad 2: KM18 -> KM14
- SW8 pad 2: KM11 -> KM17
- SW80 pad 2: KM18 -> KM15
- SW81 pad 2: KM18 -> KM15
- SW82 pad 1: GND -> Net-(D82-A)
- SW82 pad 2: SBRES -> KM18
- SW9 pad 2: KM11 -> KM17
Routing:
- net KM0: track 730.3 -> 390.9 mm, vias 4 -> 3
- net KM4: track 600.9 -> 326.2 mm, vias 4 -> 9
- net KM15: track 360.3 -> 602.8 mm, vias 3 -> 7
- net KM2: track 646.4 -> 438.5 mm, vias 4 -> 8
- net KM1: track 669.6 -> 468.9 mm, vias 4 -> 3
- net KM3: track 624.2 -> 463.3 mm, vias 4 -> 6
- net KM17: track 453.0 -> 585.9 mm, vias 7 -> 8
- net KM16: track 372.4 -> 503.4 mm, vias 3 -> 7
- net KM6: track 406.2 -> 529.5 mm, vias 3 -> 11
- net SBRES: track 384.7 -> 271.8 mm, vias 3 -> 1
- net KM10: track 358.0 -> 454.8 mm, vias 2 -> 9
- net KM13: track 325.0 -> 411.2 mm, vias 3 -> 8
- net KM9: track 410.5 -> 494.1 mm, vias 3 -> 9
- net KM12: track 301.7 -> 381.5 mm, vias 3 -> 9
- net KM7: track 408.0 -> 483.0 mm, vias 3 -> 7
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