File: keyboard/Aleste520_Keyboard.kicad_sch (KiCad schematic)
At the start: 165 parts, among them J1 X8_COLS_2x06, J2 X9_ROWS_2x06, SW1 ESC, SW10 9, SW11 0, SW12 TAB, SW13 Q, SW14 W, SW15 E, SW16 R, SW17 T, SW18 Y, SW19 U, SW2 1, SW20 I, SW21 O, SW22 P, SW23 CAPS, SW24 A, SW25 S, SW26 D, SW27 F, SW28 G, SW29 H, SW3 2, SW30 J, SW31 K, SW32 L, SW33 SEMI, SW34 SHIFT, SW35 Z, SW36 X, SW37 C, SW38 V, SW39 B, SW4 3, SW40 N, SW41 M, SW42 COMMA, SW43 DOT, SW44 SLASH, SW45 CTRL, SW46 RUS_LAT, SW47 COPY, SW48 STOP, SW49 SELECT, SW5 4, SW50 SPACE, SW51 GRAPH, SW52 CODE, SW53 MINUS, SW54 CARET, SW55 AT, SW56 F0, SW57 F1, SW58 F2, SW59 F3, SW6 5, SW60 F4, SW61 F5, SW62 F6, SW63 F7, SW64 F8, SW65 F9, SW66 FDOT, SW67 ENTER_NP, SW68 LBRACK, SW69 RBRACK, SW7 6, SW70 BSLASH, SW71 COLON, SW72 CLR, SW73 DEL, SW74 INS, SW75 HOME, SW76 END, SW77 UP, SW78 DOWN, SW79 LEFT, SW8 7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

Commit message: Feat(keyboard,case): decode RFVDKEY.BIN/AL512.BIN matrix, redesign staggered keyboard PCB with 6.25U stabilized Spacebar, and convert case to FreeCAD 1.1 (.FCStd)
Parts:
- added D82: 1N4148, Diode_THT:D_DO-35_SOD27_P7.62mm_Horizontal, symbol Device:D
- added SW83: RESET, Button_Switch_Keyboard:SW_Cherry_MX_1.00u_PCB, symbol Switch:SW_Push
- SW10: value 9 -> DEL; footprint Button_Switch_Keyboard:SW_Cherry_MX_1.00u_PCB -> Button_Switch_Keyboard:SW_Cherry_MX_1.25u_PCB
- SW11: value 0 -> 1
- SW12: value TAB -> 2
- SW13: value Q -> 3
- SW14: value W -> 4
- SW15: value E -> 5
- SW16: value R -> 6
- SW17: value T -> 7
- SW18: value Y -> 8
- SW19: value U -> 9
- SW2: value 1 -> F1_MSX; footprint Button_Switch_Keyboard:SW_Cherry_MX_1.00u_PCB -> Button_Switch_Keyboard:SW_Cherry_MX_1.25u_PCB
- SW20: value I -> 0
- SW21: value O -> MINUS
- SW22: value P -> CARET
- SW23: value CAPS -> BSLASH
- SW24: value A -> F7
- SW25: value S -> F8
- SW26: value D -> F9
- SW27: value F -> UP
- SW28: value G -> TAB; footprint Button_Switch_Keyboard:SW_Cherry_MX_1.00u_PCB -> Button_Switch_Keyboard:SW_Cherry_MX_1.50u_PCB
- SW29: value H -> Q
- SW3: value 2 -> F2_MSX; footprint Button_Switch_Keyboard:SW_Cherry_MX_1.00u_PCB -> Button_Switch_Keyboard:SW_Cherry_MX_1.25u_PCB
- SW30: value J -> W
- SW31: value K -> E
- SW32: value L -> R
- SW33: value SEMI -> T
- SW34: value SHIFT -> Y
- SW35: value Z -> U
- SW36: value X -> I
- SW37: value C -> O
- SW38: value V -> P
- SW39: value B -> AT
- SW4: value 3 -> F3_MSX; footprint Button_Switch_Keyboard:SW_Cherry_MX_1.00u_PCB -> Button_Switch_Keyboard:SW_Cherry_MX_1.25u_PCB
- SW40: value N -> LBRACK
- SW41: value M -> F4
- SW42: value COMMA -> F5
- SW43: value DOT -> F6
- SW44: value SLASH -> LEFT
- SW45: value CTRL -> CAPS; footprint Button_Switch_Keyboard:SW_Cherry_MX_1.00u_PCB -> Button_Switch_Keyboard:SW_Cherry_MX_1.75u_PCB
- SW46: value RUS_LAT -> A
- SW47: value COPY -> S
- SW48: value STOP -> D
- SW49: value SELECT -> F
- SW5: value 4 -> F4_MSX; footprint Button_Switch_Keyboard:SW_Cherry_MX_1.00u_PCB -> Button_Switch_Keyboard:SW_Cherry_MX_1.25u_PCB
- SW50: value SPACE -> G
- SW51: value GRAPH -> H
- SW52: value CODE -> J
- SW53: value MINUS -> K
- SW54: value CARET -> L
- SW55: value AT -> SEMI
- SW56: value F0 -> COLON
- SW57: value F1 -> RBRACK
- SW58: value F2 -> F1
- SW59: value F3 -> F2
- SW6: value 5 -> F5_MSX; footprint Button_Switch_Keyboard:SW_Cherry_MX_1.00u_PCB -> Button_Switch_Keyboard:SW_Cherry_MX_1.25u_PCB
- SW60: value F4 -> F3
- SW61: value F5 -> RIGHT
- SW62: value F6 -> SHIFT; footprint Button_Switch_Keyboard:SW_Cherry_MX_1.00u_PCB -> Button_Switch_Keyboard:SW_Cherry_MX_2.00u_PCB
- SW63: value F7 -> Z
- SW64: value F8 -> X
- SW65: value F9 -> C
- SW66: value FDOT -> V
- SW67: value ENTER_NP -> B
- SW68: value LBRACK -> N
- SW69: value RBRACK -> M
- SW7: value 6 -> SELECT; footprint Button_Switch_Keyboard:SW_Cherry_MX_1.00u_PCB -> Button_Switch_Keyboard:SW_Cherry_MX_1.25u_PCB
- SW70: value BSLASH -> COMMA
- SW71: value COLON -> DOT
- SW72: value CLR -> SLASH
- SW73: value DEL -> RETURN; footprint Button_Switch_Keyboard:SW_Cherry_MX_1.00u_PCB -> Button_Switch_Keyboard:SW_Cherry_MX_1.50u_PCB
- SW74: value INS -> F0
- SW75: value HOME -> FDOT
- SW76: value END -> ENTER
- SW77: value UP -> DOWN
- SW78: value DOWN -> CTRL; footprint Button_Switch_Keyboard:SW_Cherry_MX_1.00u_PCB -> Button_Switch_Keyboard:SW_Cherry_MX_1.50u_PCB
- SW79: value LEFT -> RUS_LAT; footprint Button_Switch_Keyboard:SW_Cherry_MX_1.00u_PCB -> Button_Switch_Keyboard:SW_Cherry_MX_1.25u_PCB
- SW8: value 7 -> STOP; footprint Button_Switch_Keyboard:SW_Cherry_MX_1.00u_PCB -> Button_Switch_Keyboard:SW_Cherry_MX_1.25u_PCB
- SW80: value RIGHT -> COPY; footprint Button_Switch_Keyboard:SW_Cherry_MX_1.00u_PCB -> Button_Switch_Keyboard:SW_Cherry_MX_1.25u_PCB
- SW81: value RETURN -> SPACE; footprint Button_Switch_Keyboard:SW_Cherry_MX_1.00u_PCB -> Button_Switch_Keyboard:SW_Cherry_MX_6.25u_PCB
- SW82: value RESET -> GRAPH; footprint Button_Switch_Keyboard:SW_Cherry_MX_1.00u_PCB -> Button_Switch_Keyboard:SW_Cherry_MX_1.50u_PCB
- SW9: value 8 -> CLR; footprint Button_Switch_Keyboard:SW_Cherry_MX_1.00u_PCB -> Button_Switch_Keyboard:SW_Cherry_MX_1.25u_PCB
Connections:
- net GND: now also J1.12 (Pin_12), SW83.2; no longer J1.1 (Pin_1), SW82.1
- net KM0: now also D24.1 (K), D25.1 (K), D26.1 (K), D62.1 (K), J1.10 (Pin_10); no longer D1.1 (K), D12.1 (K), D23.1 (K), D34.1 (K), D45.1 (K), D56.1 (K), D67.1 (K), D77.1 (K), J1.12 (Pin_12)
- net KM1: now also D1.1 (K), D28.1 (K), D45.1 (K), D74.1 (K), D75.1 (K), D76.1 (K), D79.1 (K); no longer D13.1 (K), D2.1 (K), D24.1 (K), D35.1 (K), D46.1 (K), D57.1 (K), D68.1 (K)
- net KM10: now also D18.1 (K), D19.1 (K), D39.1 (K), D48.1 (K), D57.1 (K), D63.1 (K), D70.1 (K), J1.1 (Pin_1); no longer D11.1 (K), D22.1 (K), D33.1 (K), D44.1 (K), D55.1 (K), J1.2 (Pin_2)
- net KM11: now also SW14.2, SW17.2, SW18.2, SW55.2; no longer SW10.2, SW11.2, SW7.2, SW8.2, SW9.2
- net KM12: now also SW11.2, SW28.2, SW31.2, SW40.2, SW52.2, SW57.2; no longer SW14.2, SW17.2, SW18.2, SW19.2, SW20.2, SW21.2, SW22.2
- net KM13: now also SW35.2, SW38.2, SW48.2, SW49.2, SW50.2, SW53.2, SW54.2, SW65.2, SW68.2, SW78.2; no longer SW23.2, SW24.2, SW25.2, SW26.2, SW27.2, SW28.2, SW29.2, SW30.2, SW31.2, SW32.2, SW33.2
- net KM14: now also SW29.2, SW30.2, SW32.2, SW46.2, SW67.2, SW79.2; no longer SW35.2, SW38.2, SW40.2, SW41.2, SW42.2, SW43.2, SW44.2
- net KM15: now also SW22.2, SW33.2, SW44.2, SW62.2, SW64.2, SW69.2, SW70.2, SW80.2, SW81.2; no longer SW46.2, SW48.2, SW49.2, SW50.2, SW51.2, SW52.2, SW53.2, SW54.2, SW55.2
- net KM16: now also SW10.2, SW23.2, SW24.2, SW41.2, SW71.2, SW74.2, SW77.2; no longer SW56.2, SW57.2, SW59.2, SW60.2, SW62.2, SW63.2, SW64.2, SW65.2
- net KM17: now also SW25.2, SW27.2, SW42.2, SW51.2, SW56.2, SW59.2, SW63.2, SW8.2, SW9.2; no longer SW67.2, SW68.2, SW69.2, SW70.2, SW71.2, SW72.2, SW74.2, SW76.2
- net KM18: now also SW19.2, SW20.2, SW21.2, SW26.2, SW43.2, SW60.2, SW7.2, SW72.2, SW76.2, SW82.2; no longer SW77.2, SW78.2, SW79.2, SW80.2, SW81.2
- net KM2: now also D29.1 (K), D49.1 (K), D52.1 (K), D55.1 (K), D59.1 (K), D60.1 (K), D80.1 (K), J1.8 (Pin_8); no longer D14.1 (K), D25.1 (K), D3.1 (K), D36.1 (K), D47.1 (K), D69.1 (K), D79.1 (K), J1.10 (Pin_10)
- net KM3: now also D11.1 (K), D2.1 (K), D22.1 (K), D34.1 (K), D41.1 (K), D42.1 (K), D43.1 (K), D65.1 (K); no longer D15.1 (K), D26.1 (K), D37.1 (K), D4.1 (K), D48.1 (K), D59.1 (K), D70.1 (K), D80.1 (K)
- net KM4: now also D12.1 (K), D3.1 (K), D30.1 (K), D35.1 (K), D47.1 (K), D9.1 (K), J1.6 (Pin_6); no longer D16.1 (K), D27.1 (K), D38.1 (K), D49.1 (K), D5.1 (K), D60.1 (K), D71.1 (K), D81.1 (K), J1.8 (Pin_8)
- net KM5: now also D10.1 (K), D13.1 (K), D4.1 (K), D46.1 (K), D53.1 (K), D69.1 (K), D7.1 (K), D8.1 (K); no longer D17.1 (K), D28.1 (K), D39.1 (K), D50.1 (K), D6.1 (K), D61.1 (K), D72.1 (K)
- net KM6: now also D14.1 (K), D31.1 (K), D36.1 (K), D38.1 (K), D61.1 (K), D81.1 (K), J1.4 (Pin_4), D82.1 (K); no longer D18.1 (K), D29.1 (K), D40.1 (K), D51.1 (K), D62.1 (K), D7.1 (K), J1.6 (Pin_6)
- net KM7: now also D15.1 (K), D27.1 (K), D32.1 (K), D33.1 (K), D5.1 (K), D68.1 (K), D72.1 (K), D77.1 (K); no longer D19.1 (K), D30.1 (K), D41.1 (K), D52.1 (K), D63.1 (K), D74.1 (K), D8.1 (K)
- net KM8: now also D16.1 (K), D21.1 (K), D37.1 (K), D50.1 (K), D56.1 (K), D6.1 (K), D71.1 (K), J1.2 (Pin_2); no longer D20.1 (K), D31.1 (K), D42.1 (K), D53.1 (K), D75.1 (K), D9.1 (K), J1.4 (Pin_4)
- net KM9: now also D17.1 (K), D20.1 (K), D23.1 (K), D40.1 (K), D44.1 (K), D51.1 (K), D67.1 (K); no longer D10.1 (K), D21.1 (K), D32.1 (K), D43.1 (K), D65.1 (K), D76.1 (K)
- net SBRES: now also SW83.1; no longer SW82.2
- new net: D82.2 (A), SW82.1
Other:
- title: Aleste 520EX Mechanical Keyboard (11x8 Matrix + 1N4148 NKRO + Reset) -> Aleste 520EX Staggered Mechanical Keyboard (82-Key Matrix + 6.25U Spacebar + Reset)
